Commit message: Restore T800 get-up reward and control contracts
Align T800 get-up with H1-style training while keeping head joints physically present but outside policy I/O. Add sole auxiliary markers so ground-parallel sampling uses actual sole points, and enable non-foot collision style penalty.

Constraint: T800 head joints must stay movable for PD locking, and collapse_fixed_joints remains disabled for auxiliary sole markers.

Rejected: Making head URDF joints fixed | this would change the asset contract and remove PD-controlled default locking.

Rejected: Sampling original ankle body with sole markers | mixed heights break the ground-parallel variance threshold.

Confidence: high

Scope-risk: moderate

Directive: Keep T800 policy dimensions at 23 controlled joints unless the observation/action contract is intentionally retrained.

Tested: py_compile for T800 config, host_ground, and test file; host conda unittest tests/test_t800_host_config.py ran 12 tests OK; git diff --cached --check.

Not-tested: Full 30000-iteration training completion; Slurm job 2386 was started separately and remains a runtime validation.

Co-authored-by: OmX <omx@oh-my-codex.dev>

File: legged_gym/resources/robots/t800_stl/urdf/serial_t800_stl.urdf (robot description, URDF)
Before this commit: robot t800, 30 links, 29 joints
Links:
- added link auxiliary_LINK_ANKLE_ROLL_L_link1; visual sphere radius=0.01
- added link auxiliary_LINK_ANKLE_ROLL_L_link2; visual sphere radius=0.01
- added link auxiliary_LINK_ANKLE_ROLL_L_link3; visual sphere radius=0.01
- added link auxiliary_LINK_ANKLE_ROLL_L_link4; visual sphere radius=0.01
- added link auxiliary_LINK_ANKLE_ROLL_R_link1; visual sphere radius=0.01
- added link auxiliary_LINK_ANKLE_ROLL_R_link2; visual sphere radius=0.01
- added link auxiliary_LINK_ANKLE_ROLL_R_link3; visual sphere radius=0.01
- added link auxiliary_LINK_ANKLE_ROLL_R_link4; visual sphere radius=0.01
Joints:
- added joint auxiliary_LINK_ANKLE_ROLL_L_joint1: type fixed, parent LINK_ANKLE_ROLL_L, child auxiliary_LINK_ANKLE_ROLL_L_link1, origin xyz=0.15 0.05 -0.06453 rpy=0 0 0
- added joint auxiliary_LINK_ANKLE_ROLL_L_joint2: type fixed, parent LINK_ANKLE_ROLL_L, child auxiliary_LINK_ANKLE_ROLL_L_link2, origin xyz=0.15 -0.05 -0.06453 rpy=0 0 0
- added joint auxiliary_LINK_ANKLE_ROLL_L_joint3: type fixed, parent LINK_ANKLE_ROLL_L, child auxiliary_LINK_ANKLE_ROLL_L_link3, origin xyz=-0.11 0.05 -0.06453 rpy=0 0 0
- added joint auxiliary_LINK_ANKLE_ROLL_L_joint4: type fixed, parent LINK_ANKLE_ROLL_L, child auxiliary_LINK_ANKLE_ROLL_L_link4, origin xyz=-0.11 -0.05 -0.06453 rpy=0 0 0
- added joint auxiliary_LINK_ANKLE_ROLL_R_joint1: type fixed, parent LINK_ANKLE_ROLL_R, child auxiliary_LINK_ANKLE_ROLL_R_link1, origin xyz=0.15 0.05 -0.06453 rpy=0 0 0
- added joint auxiliary_LINK_ANKLE_ROLL_R_joint2: type fixed, parent LINK_ANKLE_ROLL_R, child auxiliary_LINK_ANKLE_ROLL_R_link2, origin xyz=0.15 -0.05 -0.06453 rpy=0 0 0
- added joint auxiliary_LINK_ANKLE_ROLL_R_joint3: type fixed, parent LINK_ANKLE_ROLL_R, child auxiliary_LINK_ANKLE_ROLL_R_link3, origin xyz=-0.11 0.05 -0.06453 rpy=0 0 0
- added joint auxiliary_LINK_ANKLE_ROLL_R_joint4: type fixed, parent LINK_ANKLE_ROLL_R, child auxiliary_LINK_ANKLE_ROLL_R_link4, origin xyz=-0.11 -0.05 -0.06453 rpy=0 0 0
